File: lambda-x2/analog.kicad_sch (KiCad schematic)
At the start: 16 parts, among them U4 MCP6002T-I/SN

Commit message: Further updates for Rev2
Parts:
- added C77, C97: 100n, Capacitor_SMD:C_0402_1005Metric, symbol Device:C
- C2, C54: LCSC C106205 -> C1523
- R100, R101: value 160k -> 10k; LCSC C409854 -> C25744
- R98, R99: value 82k -> 5.6k; LCSC C325373 -> C25908
Connections:
- net GND: now also C77.2, C97.2
- net at D24.1 (A1), R97.2, U4.3 (+): now also C97.1
- net at D23.1 (A1), R51.2, U4.5 (+): now also C77.1
Other:
- note added: "1.56x div"
- note removed: "1.524x div"
- moved on the sheet: R51, R97
