File: lambda-x2/lsu.kicad_sch (KiCad schematic)
At the start: 51 parts, among them U12 MCP6002T-I/SN, U3 MCP6002T-I/SN, U9 GS8332-SR

Commit message: First version for lambda-x2 based on rev1
Parts:
- added C25: 100n, Capacitor_SMD:C_0402_1005Metric, symbol Device:C
- added U21: SN74HCS126PWR, Package_SO:TSSOP-14_4.4x5mm_P0.65mm, symbol 74xx_IEEE:74126
- C30, C9, R84: now not fitted
Connections:
- net +3V3: now also C25.1, U21.14 (VCC), U21.14 (VCC), U21.14 (VCC), U21.14 (VCC)
- net GND: now also C25.2, U21.7 (GND), U21.7 (GND), U21.7 (GND), U21.7 (GND)
- net Nernst_4.2_esr_drive: now also U21.13 (EN); no longer R41.2
- net Nernst_4.9_bias: now also U21.4 (EN), U21.5 (D); no longer R22.1
- net Nernst_4.9_esr_drive: now also U21.10 (EN); no longer R24.2
- net Nernst_ADV_esr_drive: now also U21.1 (EN); no longer R25.2
- new net Nernst_4.2_esr_drive_O: R41.2, U21.11 (O)
- new net Nernst_4.9_bias_O: R22.1, U21.6 (O)
- new net Nernst_4.9_esr_drive_O: R24.2, U21.8 (O)
- new net Nernst_ADV_esr_drive_O: R25.2, U21.3 (O)
- new net Nernst_drive: U21.12 (D), U21.2 (D), U21.9 (D)

Commit message: Further updates for Rev2
Parts:
- R11, R5, R7, R9: value 10k 0.1% -> 10k; footprint Resistor_SMD:R_0603_1608Metric -> Resistor_SMD:R_0402_1005Metric; LCSC C309083 -> C25744
- R12: value 47R -> 47; footprint Resistor_SMD:R_0603_1608Metric -> Resistor_SMD:R_0402_1005Metric; LCSC C328363 -> C25118
- R13: value 10k 1% -> 10k
- R15: value 2.7k 0.1% -> 2.7k; LCSC C318131 -> C13167
- R17: value 30k 1% -> 30k
- R19, R20: value 100k 0.1% -> 100k; footprint Resistor_SMD:R_0603_1608Metric -> Resistor_SMD:R_0402_1005Metric; LCSC C122538 -> C25741
- R22: value 62k 1% -> 62k
- R24: value 22k 0.1% -> 22k; footprint Resistor_SMD:R_0603_1608Metric -> Resistor_SMD:R_0402_1005Metric; LCSC C705830 -> C25768
- R25: value 47k 1% -> 47k; footprint Resistor_SMD:R_0603_1608Metric -> Resistor_SMD:R_0402_1005Metric; LCSC C25819 -> C25792
- R3: value 61.9R 1% -> 61.9; footprint Resistor_SMD:R_0805_2012Metric -> Resistor_SMD:R_0603_1608Metric; LCSC C322537 -> C23092
- R4: value 10R -> 10; footprint Resistor_SMD:R_1206_3216Metric -> Resistor_SMD:R_0402_1005Metric; LCSC C17903 -> C25077
- R41: value 6.8k 0.1% -> 6.8k; footprint Resistor_SMD:R_0603_1608Metric -> Resistor_SMD:R_0402_1005Metric; LCSC C705876 -> C25917
Other:
- moved on the sheet: R24, R25, R41
