File: lambda-x2/lambda-x2.kicad_sch (KiCad schematic)
At the start: 155 parts, among them J1 FTSH-107-01-F-DV-K, J2 tc2030-idc-nl, J3 Conn_02x02_Odd_Even, J4 Conn_01x10, P1 33311-24AW-2, Q1 BTS3028, Q2 BTS3028, Q3 BTS3028, Q4 BTS3028, U17 MCP6002T-I/SN, U18 JDY-33, U2 STM32F103RCTx, U4 LM78M05_TO252, U5 XC6206P332MR, U6 REF3033, U7 MCP6002T-I/SN, U8 TJA1051T-3, Y1 XXDCELNANF-8MHZ

Commit message: First version for lambda-x2 based on rev1
Parts:
- removed C2, C26, C55, C57: 100n, Capacitor_SMD:C_0402_1005Metric, symbol Device:C
- removed C21: 1u 25V, Capacitor_SMD:C_0603_1608Metric, symbol Device:C
- removed C22: 100n 25V, Capacitor_SMD:C_0603_1608Metric, symbol Device:C
- removed C25, C54: 1u, Capacitor_SMD:C_0402_1005Metric, symbol Device:C
- removed C70, C71: 20pF 50V, Capacitor_SMD:C_0402_1005Metric, symbol Device:C
- removed C77, C78: 1n, Capacitor_SMD:C_0402_1005Metric, symbol Device:C
- removed D23, D24: ESD5V0D9B, Diode_SMD:D_SOD-923, symbol Diode:ESD9B5.0ST5G
- removed D6: 1N4148W, Diode_SMD:D_SOD-123, symbol Diode:1N4148W
- removed J1: FTSH-107-01-F-DV-K, Connector_PinHeader_1.27mm:PinHeader_2x07_P1.27mm_Vertical_SMD, symbol Connector_Generic:Conn_02x07_Odd_Even
- removed JP1: SolderJumper_2_Open, Jumper:SolderJumper-2_P1.3mm_Open_TrianglePad1.0x1.5mm, symbol Jumper:SolderJumper_2_Open
- removed R100, R101: 160k, Resistor_SMD:R_0402_1005Metric, symbol Device:R
- removed R112, R96, R97: 10k, Resistor_SMD:R_0402_1005Metric, symbol Device:R
- removed R40, R46, R50, R51: 1K, Resistor_SMD:R_0603_1608Metric, symbol Device:R
- removed R98, R99: 82k, Resistor_SMD:R_0402_1005Metric, symbol Device:R
- removed U17: MCP6002T-I/SN, Package_SO:SOIC-8_3.9x4.9mm_P1.27mm, symbol Amplifier_Operational:MCP6002-xSN
- removed U4: LM78M05_TO252, Package_TO_SOT_SMD:TO-252-2, symbol Regulator_Linear:LM78M05_TO252
- removed U5: XC6206P332MR, Package_TO_SOT_SMD:SOT-23, symbol Regulator_Linear:XC6206PxxxMR
- removed Y1: XXDCELNANF-8MHZ, Crystal:Crystal_SMD_3225-4Pin_3.2x2.5mm, symbol Device:Crystal_Small
- added C21, C22: 33p, Capacitor_SMD:C_0402_1005Metric, symbol Device:C_Small
- added C81: 4.7u, Capacitor_SMD:C_0805_2012Metric, symbol Device:C
- added C82: 56u, Capacitor_THT:CP_Radial_D8.0mm_P3.50mm, symbol proteus-rescue:CP-Device
- added C83, C90, C91, C92, C93: 10u, Capacitor_SMD:C_1206_3216Metric, symbol Device:C
- added C84, C85: 2.2u, Capacitor_SMD:C_1206_3216Metric, symbol Device:C
- added C86: 100n, Capacitor_SMD:C_0603_1608Metric, symbol Device:C
- added C87: 10n, Capacitor_SMD:C_0603_1608Metric, symbol Device:C
- added C88: 100n, Capacitor_SMD:C_0603_1608Metric, symbol Device:C_Small
- added C89: 330p, Capacitor_SMD:C_0402_1005Metric, symbol Device:C
- added C95: 1u, Capacitor_SMD:C_0402_1005Metric, symbol Device:C
- added C96: 100n, Capacitor_SMD:C_0402_1005Metric, symbol Device:C
- added D31, D6: D_Schottky, Diode_SMD:D_SMA, symbol Device:D_Schottky
- added J5: Conn_02x05_Odd_Even, Connector_PinHeader_2.54mm:PinHeader_2x05_P2.54mm_Vertical, symbol Connector_Generic:Conn_02x05_Odd_Even
- added JP4, JP5: SolderJumper_2_Open, Jumper:SolderJumper-2_P1.3mm_Open_TrianglePad1.0x1.5mm, symbol Jumper:SolderJumper_2_Open
- added L6: 2.2u, Inductor_SMD:L_1210_3225Metric, symbol Device:L
- added L7: 10u, sunlord-MWSA0503:MWSA0503, symbol Device:L
- added R116: 1, Resistor_SMD:R_0402_1005Metric, symbol Device:R
- added R117: 10k, Resistor_SMD:R_0402_1005Metric, symbol Device:R
- added R118: 12k, Resistor_SMD:R_0402_1005Metric, symbol Device:R
- added R119: 68k, Resistor_SMD:R_0402_1005Metric, symbol Device:R
- added R120, R132, R133, R134, R135, R136, R137, R142, R143, R144: 0, Resistor_SMD:R_0402_1005Metric, symbol Device:R
- added R121, R122: 100k, Resistor_SMD:R_0402_1005Metric, symbol Device:R
- added U19: LMR14020, Package_SO:SOIC-8-1EP_3.9x4.9mm_P1.27mm_EP2.29x3mm, symbol lmr14020:LMR14020
- added U20: AMS1117-3.3, Package_TO_SOT_SMD:SOT-223-3_TabPin2, symbol Regulator_Linear:AMS1117-3.3
- added U23: TLS115, Package_SO:Infineon_PG-DSO-8-43, symbol infineon_psu:TLS115
- added Y2: 8MHz, Crystal:Crystal_SMD_5032-2Pin_5.0x3.2mm, symbol Device:Crystal
- C10, C35: value 1n -> 1u; LCSC C106205 -> C52923
- C27: value 100n -> 4.7u; footprint Capacitor_SMD:C_0402_1005Metric -> Capacitor_SMD:C_0603_1608Metric; LCSC C1525 -> C19666; LCSC_ext (none) -> 0
- C28: value 1u -> 100n; footprint Capacitor_SMD:C_0402_1005Metric -> Capacitor_SMD:C_0603_1608Metric; LCSC C52923 -> C14663; LCSC_ext (none) -> 0
- C44, C45: value 47p -> 1u; footprint Capacitor_SMD:C_0402_1005Metric -> Capacitor_SMD:C_0603_1608Metric; LCSC C1567 -> C15849; LCSC_ext (none) -> 0
- L5, R39: now not fitted
- Q1, Q2, Q3, Q4: value BTS3028 -> VND7NV04TR-E; footprint Package_TO_SOT_SMD:TO-252-2 -> Package_TO_SOT_SMD:TO-252-3_TabPin2; JLCPosOffset (none) -> 2,0; LCSC C112639 -> C262999
- R113: value 0R -> 10k; LCSC C325377 -> C25744; now in the parts list
- R48: footprint Resistor_SMD:R_1206_3216Metric -> Resistor_SMD:R_0603_1608Metric; LCSC C176250 -> C22787; now in the parts list
- U8: LCSC C38695 -> C6952
Connections:
- net +3V3: now also J5.1 (Pin_1), R120.2, R122.2, U20.2 (VO); no longer U8.5 (VIO)
- net +5V: now also C89.1, C90.1, C91.1, C92.1, C93.1, L7.2, R119.2, R142.1, U20.3 (VI), U23.5 (ADJ)
- net CAN_H: no longer C44.2
- net CAN_L: now also JP4.2 (B); no longer C45.1, R48.2
- net GND: now also C44.2, R113.1, R88.2, C21.2, C22.2, C81.2, C82.2, C83.2, C84.2, C85.2, C86.2, C87.2, C90.2, C91.2, C92.2, C93.2, C95.2, C96.2, D31.2 (A), J5.3 (Pin_3), J5.5 (Pin_5), J5.9 (Pin_9), R117.2, R118.2, R121.2, U19.7 (GND), U19.9 (GND), U20.1 (GND), U23.3 (GND), U23.9 (GND); no longer C44.1, R113.2, R88.1
- net L_OUT_en: now also R88.1; no longer R88.2
- net L_OUT_sense: now also R132.2, R136.2; no longer C75.1, R102.2, R105.2
- net Nernst_4.9_bias: now also R113.2
- net R_OUT_sense: now also R133.2, R137.2; no longer C76.1, R103.2, R106.2
- net SWCLK: now also J5.4 (Pin_4), R121.1
- net SWDIO: now also J5.2 (Pin_2), R122.1
- net VDDA: now also C95.1, C96.1
- net Vout1: now also JP5.1 (A), R134.1, R143.1; no longer R31.2, R32.2
- net Vout2: now also R135.1, R144.1; no longer R35.2, R37.2
- net nRESET: now also J5.10 (Pin_10)
- net 12v_PROT: now reaches TP27.1
- net 12v_PROT: now also C44.1, D6.1 (K), L6.1, R116.1, U23.7 (EN), U23.8 (IN)
- net at D4.1 (A1), F1.1, R27.1: now also D6.2 (A)
- net at U2.6 (PD1): now also C22.1, Y2.2
- net at U2.5 (PD0): now also C21.1, Y2.1
- net SWO: no longer names the net of J2.6 (SWO)
- net config1 renamed Nernst_drive
- net Nernst_drive: no longer R113.1
- new net: R134.2, R31.2, R32.2
- new net: R135.2, R35.2, R37.2
- new net: R120.1, U8.5 (VIO)
- new net: R117.1, U19.4 (RT)
- new net: C89.2, R118.1, R119.1, U19.5 (FB)
- new net: C75.1, R102.2, R105.2, R136.1
- new net: C88.1, U19.1 (BOOT)
- new net: C87.1, U19.6 (SS)
- new net: C88.2, D31.1 (K), L7.1, U19.8 (SW)
- new net: C76.1, R103.2, R106.2, R137.1
- new net: C81.1, R116.2
- new net: JP4.1 (A), R48.2
- new net 5V_SENSOR: C45.1, JP5.2 (B), R142.2, U23.1 (OUT)
- new net Dual AUX analog input 2/AIN_1: R143.2
- new net Dual AUX analog input 2/AIN_2: R144.2
- new net Dual AUX analog input 2/AOUT_1: R132.1
- new net Dual AUX analog input 2/AOUT_2: R133.1
- new net VIN: C82.1, C83.1, C84.1, C85.1, C86.1, L6.2, U19.2 (VIN), U19.3 (EN)
Other:
- added sheet Dual AUX analog input 1 (analog.kicad_sch)
- added sheet Dual AUX analog input 2 (analog.kicad_sch)
- sheet LSU analog left ports: added Nernst_drive; removed none
- sheet LSU analog right ports: added Nernst_drive; removed none
- note added: "3.3v Supply"
- note added: "5V Sensor Tracker 1 (optional)"
- note added: "Analog inputs"
- note added: "Analog reference voltage"
- note added: "Bluetooth"
- note added: "Cortex Debug Header"
- note added: "DNP for 4 analog inputs variant"
- note added: "Input Filter & 5v Regulator"
- note added: "Place for 4 analog inputs variant"
- note added: "TJA1050 (which is LCSC basic part) can be used as drop-in replacement: RXD connected to MCU PA11 (5V tolerant) TJA1050 has logic HIGH-level input voltage of 2.0V at TXD DNP 0R Resistor on VIO in this case!"
- note added: "Tie BOOT1 to GND to resolve "DFU mode/floating PB2""
- note removed: "1.524x div"
- note removed: "2x analog inputs"
- note removed: "Debug"
- note removed: "n.p."
- note removed: "reg 35V max Vin"
- moved on the sheet: C1, C12, C19, C32, C33, C34, C36, C38, C39, C4, C40, C41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

Commit message: Further updates for Rev2
Parts:
- removed JP2, JP3: SolderJumper_2_Open, Jumper:SolderJumper-2_P1.3mm_Open_TrianglePad1.0x1.5mm, symbol Jumper:SolderJumper_2_Open
- added C100, C101, C102, C99: 10u, Capacitor_SMD:C_0805_2012Metric, symbol Device:C
- added C78: 100n, Capacitor_SMD:C_0402_1005Metric, symbol Device:C
- added R138: 10k, Resistor_SMD:R_0402_1005Metric, symbol Device:R
- added R139: 0, Resistor_SMD:R_0402_1005Metric, symbol Device:R
- added U17: TPS3823, Package_TO_SOT_SMD:SOT-23-5, symbol MAX823:MAX823
- C27: value 4.7u -> 10u; footprint Capacitor_SMD:C_0603_1608Metric -> Capacitor_SMD:C_0805_2012Metric; LCSC C19666 -> C440198
- C72, C75, C76, C79, C80: LCSC C106205 -> C1523
- C81: footprint Capacitor_SMD:C_0805_2012Metric -> Capacitor_SMD:C_1206_3216Metric; LCSC C98192 -> C29823
- C82: now not fitted; now left out of the parts list
- C83: footprint Capacitor_SMD:C_1206_3216Metric -> Capacitor_SMD:C_0805_2012Metric; LCSC C13585 -> C440198
- C84, C85: footprint Capacitor_SMD:C_1206_3216Metric -> Capacitor_SMD:C_0805_2012Metric; LCSC C170101 -> C377773
- D12: value NUP2105L -> PSM712-LF-T7; LCSC C284104 -> C32677; LCSC_alt (none) -> C284104 (NUP2105L)
- J2, U18: LCSC (none) -> N/A
- JP4, P1: now left out of the parts list
- L5: value 470R@100MHz -> 600R@100MHz; LCSC C97853 -> C1002
- R102, R103, R27, R52, R81: value 100k 1% -> 100k; footprint Resistor_SMD:R_0603_1608Metric -> Resistor_SMD:R_0402_1005Metric; LCSC C217279 -> C25741
- R105, R106, R36, R53, R82: value 10k 1% -> 10k
- R114, R115: LCSC C328363 -> C23182; now not fitted
- R116: footprint Resistor_SMD:R_0402_1005Metric -> Resistor_SMD:R_0603_1608Metric; LCSC C25086 -> C22936
- R2, R6: value 10k 0.1% -> 1k; footprint Resistor_SMD:R_0603_1608Metric -> Resistor_SMD:R_0402_1005Metric; LCSC C309083 -> C11702
- R30, R80, R88, R89: LCSC C11702 -> C25744
- R31, R35: value 330R -> 330
- R32: value 82k -> 5.6k; LCSC C325373 -> C25908
- R33, R38: value 160k -> 10k; LCSC C409854 -> C25744
- R37: value 82k -> 5.6k; LCSC C23254 -> C25908
- R48: value 120R -> 120
- SW1, SW2: value ~ -> SW_Push; footprint Button_Switch_SMD:SW_SPST_CK_RS282G05A3 -> Button_Switch_SMD:SW_SPST_EVQQ2; LCSC C398054 -> C318884; LCSC_ext (none) -> 1; now in the parts list
- U23: LCSC N/A -> C3743696
Connections:
- net +3V3: now also SW2.1, R138.2, U17.5 (VCC); no longer SW2.2
- net Boot0: now also SW2.2; no longer SW2.1
- net GND: now also C100.2, C101.2, C102.2, C78.2, C99.2, U17.2 (GND)
- net VIN: now also C100.1, C101.1, C102.1, C99.1
- net nRESET: now also C78.1, R138.1, R139.1, U17.1 (~{RESET}); no longer SW1.2
- new net: R139.2, SW1.2, U17.3 (~{MR})
Other:
- added sheet EGT Protection (egt-prot.kicad_sch)
- note added: "1.593x gain"
- note added: "Basic part but only 12V"
- note added: "Remove if used"
- note removed: "1.524x gain"
- moved on the sheet: C44, C45, C7, C81, D5, L6, R116, R142, R2, R6, U23

Commit message: minor rework
Parts:
- C10, C35: value 1u -> 1n; LCSC C52923 -> C1523
- D2, D29, D30, D5: LCSC C72043 -> C2986059
- L6: value 2.2u -> 2.2u -> 1.5u; LCSC C36828 -> C394996; LCSC_ext 1 -> C36828
- Q1, Q2, Q3, Q4: JLCRotOffset (none) -> 180
- U2: LCSC_alt (none) -> C8322
Changed lines of the file:
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@@
   (junction (at 222.25 231.775) (diameter 0) (color 0 0 0 0)
   )
+  (junction (at 228.6 257.175) (diameter 0) (color 0 0 0 0)
+  )
   (junction (at 487.68 175.26) (diameter 0) (color 0 0 0 0)
   )
@@
   (junction (at 315.595 34.29) (diameter 0) (color 0 0 0 0)
   )
+  (junction (at 228.6 231.775) (diameter 0) (color 0 0 0 0)
+  )
   (junction (at 173.99 388.62) (diameter 0) (color 0 0 0 0)
   )
@@
   (junction (at 215.265 207.01) (diameter 0) (color 0 0 0 0)
   )
-  (junction (at 228.6 231.775) (diameter 0) (color 0 0 0 0)
-  )
   (junction (at 296.545 34.29) (diameter 0) (color 0 0 0 0)
   )
@@
   (junction (at 550.545 40.005) (diameter 0) (color 0 0 0 0)
   )
-  (junction (at 228.6 257.175) (diameter 0) (color 0 0 0 0)
-  )
   (junction (at 254 313.055) (diameter 0) (color 0 0 0 0)
   )
@@
     (stroke (width 0) (type default))
   )
-  (wire (pts (xy 228.6 257.175) (xy 234.95 257.175))
-    (stroke (width 0) (type default))
-  )
   (wire (pts (xy 176.53 264.795) (xy 179.07 264.795))
     (stroke (width 0) (type default))
@@
     (stroke (width 0) (type default))
   )
-  (wire (pts (xy 222.25 231.775) (xy 228.6 231.775))
-    (stroke (width 0) (type default))
-  )
   (wire (pts (xy 247.65 76.2) (xy 247.65 77.47))
     (stroke (width 0) (type default))
@@
     (stroke (width 0) (type default))
   )
+  (wire (pts (xy 228.6 257.175) (xy 234.95 257.175))
+    (stroke (width 0) (type default))
+  )
   (wire (pts (xy 527.558 130.048) (xy 527.558 130.683))
     (stroke (width 0) (type default))
@@
     (stroke (width 0) (type default))
   )
+  (wire (pts (xy 228.6 231.775) (xy 234.95 231.775))
+    (stroke (width 0) (type default))
+  )
   (wire (pts (xy 224.79 365.76) (xy 234.95 365.76))
     (stroke (width 0) (type default))
@@
     (stroke (width 0) (type default))
   )
-  (wire (pts (xy 228.6 231.775) (xy 234.95 231.775))
+  (wire (pts (xy 222.25 231.775) (xy 228.6 231.775))
     (stroke (width 0) (type default))
   )
@@
       (effects (font (size 1.27 1.27)) hide)
     )
-    (property "LCSC" "C72043" (at 550.545 134.62 0)
+    (property "LCSC" "C2986059" (at 550.545 134.62 0)
       (effects (font (size 1.27 1.27)) hide)
     )
@@
       (effects (font (size 1.27 1.27)) hide)
     )
-    (property "LCSC" "C72043" (at 527.558 134.493 0)
+    (property "LCSC" "C2986059" (at 527.558 134.493 0)
       (effects (font (size 1.27 1.27)) hide)
     )
@@
       (effects (font (size 1.27 1.27)) hide)
     )
+    (property "JLCRotOffset" "180" (at 171.45 264.795 0)
+      (effects (font (size 1.27 1.27)) hide)
+    )
     (pin "1")
     (pin "2")
@@
       (effects (font (size 1.27 1.27)) hide)
     )
-    (property "LCSC" "C72043" (at 521.335 313.69 0)
+    (property "LCSC" "C2986059" (at 521.335 313.69 0)
       (effects (font (size 1.27 1.27)) hide)
     )
@@
       (effects (font (size 1.27 1.27)) hide)
     )
+    (property "JLCRotOffset" "180" (at 171.45 187.96 0)
+      (effects (font (size 1.27 1.27)) hide)
+    )
     (pin "1")
     (pin "2")
@@
       (effects (font (size 1.27 1.27)) hide)
     )
+    (property "JLCRotOffset" "180" (at 171.45 239.395 0)
+      (effects (font (size 1.27 1.27)) hide)
+    )
     (pin "1")
     (pin "2")
@@
       (effects (font (size 1.27 1.27)) hide)
     )
+    (property "LCSC_alt" "C8322" (at 394.97 236.22 0)
+      (effects (font (size 1.27 1.27)) hide)
+    )
     (pin "1")
     (pin "10")
@@
       (effects (font (size 1.27 1.27)) hide)
     )
-    (property "LCSC" "C72043" (at 561.975 134.62 0)
+    (property "LCSC" "C2986059" (at 561.975 134.62 0)
       (effects (font (size 1.27 1.27)) hide)
     )
@@
       (effects (font (size 1.27 1.27)))
     )
-    (property "Value" "2.2u" (at 302.895 31.75 90)
+    (property "Value" "2.2u -> 1.5u" (at 302.895 31.75 90)
       (effects (font (size 1.27 1.27)))
     )
@@
       (effects (font (size 1.27 1.27)) hide)
     )
-    (property "LCSC" "C36828" (at 302.26 34.29 0)
+    (property "LCSC" "C394996" (at 302.26 34.29 0)
       (effects (font (size 1.27 1.27)) hide)
     )
-    (property "LCSC_ext" "1" (at 302.26 34.29 0)
+    (property "LCSC_ext" "C36828" (at 302.26 34.29 0)
       (effects (font (size 1.27 1.27)) hide)
     )
@@
       (effects (font (size 1.27 1.27)) hide)
     )
-    (pin "1")
-    (pin "2")
-    (pin "3")
-    (instances
-      (project "lambda-x2"
-        (path "/3993c707-5291-41b6-83c0-d1c09cb3833a"
-          (reference "Q4") (unit 1)
-        )
-      )
-    )
-  )
-  (symbol (lib_id "Device:C") (at 228.6 260.985 0) (unit 1)
-    (in_bom yes) (on_board yes) (dnp no)
-    (property "Reference" "C10" (at 231.521 259.8166 0)
-      (effects (font (size 1.27 1.27)) (justify left))
-    )
-    (property "Value" "1u" (at 231.521 262.128 0)
-      (effects (font (size 1.27 1.27)) (justify left))
-    )
-    (property "Footprint" "Capacitor_SMD:C_0402_1005Metric" (at 229.5652 264.795 0)
-      (effects (font (size 1.27 1.27)) hide)
-    )
-    (property "Datasheet" "~" (at 228.6 260.985 0)
-      (effects (font (size 1.27 1.27)) hide)
-    )
-    (property "LCSC" "C52923" (at 228.6 260.985 0)
+    (property "JLCRotOffset" "180" (at 171.45 214.63 0)
       (effects (font (size 1.27 1.27)) hide)
     )
     (pin "1")
     (pin "2")
+    (pin "3")
     (instances
       (project "lambda-x2"
         (path "/3993c707-5291-41b6-83c0-d1c09cb3833a"
-          (reference "C10") (unit 1)
+          (reference "Q4") (unit 1)
         )
       )
@@
     )
   )
+  (symbol (lib_id "Device:C") (at 228.6 260.985 0) (mirror y) (unit 1)
+    (in_bom yes) (on_board yes) (dnp no)
+    (property "Reference" "C10" (at 233.68 258.445 0)
+      (effects (font (size 1.27 1.27)) (justify left))
+    )
+    (property "Value" "1n" (at 236.22 262.255 0)
+      (effects (font (size 1.27 1.27)) (justify left))
+    )
+    (property "Footprint" "Capacitor_SMD:C_0402_1005Metric" (at 227.6348 264.795 0)
+      (effects (font (size 1.27 1.27)) hide)
+    )
+    (property "Datasheet" "~" (at 228.6 260.985 0)
+      (effects (font (size 1.27 1.27)) hide)
+    )
+    (property "LCSC" "C1523" (at 228.6 260.985 0)
+      (effects (font (size 1.27 1.27)) hide)
+    )
+    (pin "1")
+    (pin "2")
+    (instances
+      (project "lambda-x2"
+        (path "/3993c707-5291-41b6-83c0-d1c09cb3833a"
+          (reference "C10") (unit 1)
+        )
+      )
+    )
+  )
+  (symbol (lib_id "Device:C") (at 228.6 235.585 0) (mirror y) (unit 1)
+    (in_bom yes) (on_board yes) (dnp no)
+    (property "Reference" "C35" (at 233.68 233.045 0)
+      (effects (font (size 1.27 1.27)) (justify left))
+    )
+    (property "Value" "1n" (at 236.22 236.855 0)
+      (effects (font (size 1.27 1.27)) (justify left))
+    )
+    (property "Footprint" "Capacitor_SMD:C_0402_1005Metric" (at 227.6348 239.395 0)
+      (effects (font (size 1.27 1.27)) hide)
+    )
+    (property "Datasheet" "~" (at 228.6 235.585 0)
+      (effects (font (size 1.27 1.27)) hide)
+    )
+    (property "LCSC" "C1523" (at 228.6 235.585 0)
+      (effects (font (size 1.27 1.27)) hide)
+    )
+    (pin "1")
+    (pin "2")
+    (instances
+      (project "lambda-x2"
+        (path "/3993c707-5291-41b6-83c0-d1c09cb3833a"
+          (reference "C35") (unit 1)
+        )
+      )
+    )
+  )
   (symbol (lib_id "Jumper:SolderJumper_2_Open") (at 95.25 114.3 0) (unit 1)
     (in_bom no) (on_board yes) (dnp no)
@@
         )
       )
-    )
-  )
-  (symbol (lib_id "Device:C") (at 228.6 235.585 0) (unit 1)
-    (in_bom yes) (on_board yes) (dnp no)
-    (property "Reference" "C35" (at 231.521 234.4166 0)
-      (effects (font (size 1.27 1.27)) (justify left))
-    )
-    (property "Value" "1u" (at 231.521 236.728 0)
-      (effects (font (size 1.27 1.27)) (justify left))
-    )
-    (property "Footprint" "Capacitor_SMD:C_0402_1005Metric" (at 229.5652 239.395 0)
-      (effects (font (size 1.27 1.27)) hide)
-    )
-    (property "Datasheet" "~" (at 228.6 235.585 0)
-      (effects (font (size 1.27 1.27)) hide)
-    )
-    (property "LCSC" "C52923" (at 228.6 235.585 0)
-      (effects (font (size 1.27 1.27)) hide)
-    )
-    (pin "1")
-    (pin "2")
-    (instances
-      (project "lambda-x2"
-        (path "/3993c707-5291-41b6-83c0-d1c09cb3833a"
-          (reference "C35") (unit 1)
-        )
-      )
